File: RemoteSwitchController/remoteserialcontroller.brd (EAGLE design)
At the start: 100 x 50 mm, 37 parts, among them J1 ZX62R-AB-5P, J2 D-SUB9, Q2 MMSS8050-L, Q3 MMSS8050-L, SW1 SKRPACE010, SW2 SKRPACE010, U1 ADM3202ARUZ, U2 ESP-WROOM-32, U21 FT232RL

Commit message: [add] temporrary
Parts:
- removed C1, C11, C2, C3, C9: 0.1uF, taki-library:C0603
- removed J2: D-SUB9, taki-library:D-SUB9/C-00645/AKIZUKI
- removed U1: ADM3202ARUZ, taki-library:TSSOP16-AD
- added Q1, Q4, Q5, Q6: BSS138, taki-library:SOT23-N-MOSFET
- added R11, R12, R13, R14, R15, R16: 10k, taki-library:R0603
- R10, R9: value 100 -> 10k
- moved R10 140.9 mm to (2.54, -94.0), turned to 0 degrees
- moved R9 136.9 mm to (2.54, -87.6), turned to 0 degrees
- moved SP1 71.0 mm to (34.3, -34.3)
- moved C5 68.9 mm to (17.8, -74.9)
- moved J1 63.7 mm to (6.35, -52.1), turned to 0 degrees
- moved LED2 56.3 mm to (40.6, -62.2)
- moved R46 55.8 mm to (55.9, -61.0)
- moved LED6 55.3 mm to (45.7, -62.2)
- moved R1 54.9 mm to (33.0, -68.6)
- moved R2 54.9 mm to (36.8, -68.6)
- moved C4 54.6 mm to (11.4, -74.9)
- moved LED1 54.5 mm to (35.6, -62.2)
- moved C13 53.2 mm to (24.1, -74.9)
- moved C6 53.1 mm to (27.9, -62.2)
- moved R32 44.9 mm to (50.8, -61.0)
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Connections:
- removed net EXT_RXD: J2.2, R9.2
- removed net EXT_TXD: J2.3, R10.2
- removed net N$1: J2.1, J2.4
- removed net N$13: C1.1, U1.3
- removed net N$15: C2.1, U1.5
- removed net N$17: C11.2, U1.6
- removed net N$2: R9.1, U1.14
- new net +5V: R10.2, R12.2, R14.2, R16.2
- new net SERVO_IN_1: Q1.S, R9.1
- new net SERVO_IN_2: Q4.S, R11.1
- new net SERVO_IN_3: Q5.S, R13.1
- new net SERVO_IN_4: Q6.S, R15.1
- net +3V3: now also Q1.G, Q4.G, Q5.G, Q6.G, R11.2, R13.2, R15.2, R9.2; no longer C3.1, C9.1, U1.16
- net GND: no longer C11.1, C3.2, U1.15
- net N$11: now also Q4.D, R12.1; no longer C1.2, U1.1
- net N$14: now also Q5.D, R14.1; no longer C2.2, U1.4
- net N$16: now also Q6.D, R16.1; no longer C9.2, U1.2
- net N$3: now also Q1.D; no longer U1.13
- net RXD: no longer U1.12
- net TXD: no longer U1.11
Routing:
- net GND: track 16.7 -> 0.00 mm
- net EXT_TXD: track 12.4 -> 0.00 mm
- net N$1: track 12.3 -> 0.00 mm
- net EXT_RXD: track 9.50 -> 0.00 mm
- net N$16: track 7.51 -> 0.00 mm
- net N$13: track 4.15 -> 0.00 mm
- net N$15: track 3.96 -> 0.00 mm
- net +3V3: track 3.77 -> 0.00 mm
- net N$3: track 2.55 -> 0.00 mm
- net N$2: track 2.55 -> 0.00 mm
- net N$17: track 2.20 -> 0.00 mm
- net N$11: track 1.53 -> 0.00 mm
- net N$14: track 1.49 -> 0.00 mm
Other:
- board size 100 x 50 mm -> 160 x 100 mm
