File: RemoteSwitchController/remoteserialcontroller.brd (EAGLE design)
At the start: 73 x 22.8 mm, 35 parts, among them J1 ZX62R-AB-5P, J2 S3B-PH-K-S, J3 S3B-PH-K-S, J4 S3B-PH-K-S, J5 S3B-PH-K-S, Q1 BSS138, Q2 BSS138, Q3 BSS138, Q4 BSS138, Q5 BSS138, Q6 BSS138, U2 ESP-WROOM-32, U3 ADP3338AKCZ-3.3, U4 CP2104

Commit message: [update]update schematic and add BOM
Parts:
- added J6: S2B-PH-K-S, taki-library:S2B-PH-K-S
- added R11, R12, R13, R14: 10k, taki-library:R0603
- moved R10 30.5 mm to (70.0, 8.90), turned to 180 degrees
- moved Q6 26.0 mm to (66.1, 9.40), turned to 0 degrees
- moved Q4 24.5 mm to (55.9, 9.30), turned to 270 degrees
- moved R6 23.2 mm to (69.6, 13.6)
- moved R4 20.6 mm to (58.6, 9.40)
- moved Q5 19.4 mm to (67.0, 13.3), turned to 0 degrees
- moved Q3 18.0 mm to (53.0, 13.4), turned to 0 degrees
- moved R2 15.8 mm to (56.0, 14.0), turned to 0 degrees
Connections:
- new net N$1: Q3.G, R11.1
- new net N$2: Q5.G, R12.1
- new net N$3: Q6.G, R13.1
- new net N$4: Q4.G, R14.1
- net +5V: now also J6.1
- net GND: now also J6.2
- net SERVO1: now also R11.2; no longer Q3.G
- net SERVO2: now also R14.2; no longer Q4.G
- net SERVO3: now also R12.2; no longer Q5.G
- net SERVO4: now also R13.2; no longer Q6.G
Routing:
- net GND: track 86.9 -> 210.7 mm, vias 6 -> 155
- net +5V: track 19.7 -> 105.5 mm, vias 2 -> 6
- net SERVO4: track 0.00 -> 65.0 mm, vias 0 -> 2
- net SERVO3: track 0.00 -> 54.3 mm, vias 0 -> 2
- net SERVO2: track 0.00 -> 45.4 mm, vias 0 -> 2
- net SERVO1: track 0.00 -> 43.9 mm, vias 0 -> 2
- net +3V3: track 84.6 -> 93.5 mm, vias 4 -> 5
- net CH4: track 0.00 -> 8.81 mm
- net CH3: track 0.00 -> 6.26 mm
- net CH2: track 0.00 -> 6.00 mm
- net N$2: track 0.00 -> 5.23 mm
- net CH1: track 0.00 -> 4.47 mm
- net N$4: track 0.00 -> 2.77 mm
- net N$3: track 0.00 -> 2.18 mm
- net N$1: track 0.00 -> 1.87 mm
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- added copper zone on layer 1, net GND
- added copper zone on layer 16, net GND
