File: RemoteSerialController/remoteserialcontroller.brd (EAGLE design)
At the start: 100 x 50 mm, 37 parts, among them J1 ZX62R-AB-5P, J2 D-SUB9, Q2 MMSS8050-L, Q3 MMSS8050-L, SW1 SKRPACE010, SW2 SKRPACE010, U1 ADM3202ARUZ, U2 ESP-WROOM-32, U21 FT232RL

Commit message: [fin]finish design
Parts:
- removed C10, C8: 1000pF, taki-library:C0603
- removed J2: D-SUB9, taki-library:D-SUB9/C-00645/AKIZUKI
- removed LED1: RX, taki-library:CHIPLED_0603
- removed LED2: TX, taki-library:CHIPLED_0603
- removed LED6: LED1, taki-library:CHIPLED_0603
- removed Q3: MMSS8050-L, taki-library:SOT23
- removed R32, R46: 1k, taki-library:R0603
- removed SW1, SW2: SKRPACE010, taki-library:SKRPACE010
- removed U21: FT232RL, taki-library:SSOP28
- added C12, C15: 0.1uF, taki-library:C0603
- added C14: 5uF, taki-library:C0603
- added D1, D2, D3, D4: B, taki-library:CHIPLED_0603
- added EN, IO0: SKRPACE010, taki-library:SKRPACE010
- added J3: DM3AT-SF-PEJM5, taki-library:DM3AT-SF-PEJM5
- added J4: XM3B-0942-132L, taki-library:XM3B-0942-132L
- added Q1: BSS138, taki-library:SOT23-N-MOSFET
- added R11, R12, R13, R14, R15, R24: 10k, taki-library:R0603
- added R16: 1k, taki-library:R0603
- added U3: ADP3338AKCZ-3.3, taki-library:SOT233
- added U4: CP2104, taki-library:QFN24-SILABS
- C13: value 0.1uF -> 4.7uF
- C4: value 0.1uF -> 1uF
- Q2: value MMSS8050-L -> BSS138; device taki-library:SOT23 -> taki-library:SOT23-N-MOSFET
- R4, R6: value 470 -> 1k
- R7: value 10k -> 24k
- R8: value 10k -> 47k
- moved SP1 121.0 mm to (59.0, 9.17), turned to 90 degrees
- moved C7 117.0 mm to (37.7, 33.8), turned to 270 degrees
- moved R5 115.4 mm to (46.7, 38.8), turned to 90 degrees
- moved R3 112.4 mm to (37.7, 36.8), turned to 90 degrees
- moved R6 86.7 mm to (41.5, 5.70), turned to 90 degrees
- moved R7 82.8 mm to (37.6, 27.5), turned to 90 degrees
- moved R8 81.6 mm to (39.7, 27.5), turned to 270 degrees
- moved Q2 80.3 mm to (43.8, 35.9), turned to 270 degrees
- moved C13 75.5 mm to (48.3, 32.5), turned to 90 degrees
- moved R4 74.4 mm to (44.5, 5.70), turned to 90 degrees
- moved R2 65.4 mm to (59.9, 22.4)
- moved C6 57.9 mm to (49.5, 41.1), turned to 90 degrees
- moved C4 55.0 mm to (42.3, 26.9), turned to 180 degrees
- moved C5 53.1 mm to (52.1, 42.0), turned to 90 degrees
- moved R1 48.5 mm to (47.5, 5.70), turned to 90 degrees
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Connections:
- removed net D1_M: J1.D-, U21.16
- removed net D1_P: J1.D+, U21.15
- removed net N$10: Q3.B, R8.1
- removed net N$12: C10.2, R6.1, SW2.S1, SW2.S2
- removed net N$50: LED6.C, U2.8
- removed net N$84: C13.1, U21.17, U21.4
- removed net N$85: C4.1, J1.VCC, U21.20
- removed net SCL: U2.36
- removed net SDA: U2.33
- removed net SQW: U2.6
- removed net SW3: U2.11
- removed net SW4: U2.12
- removed net SW5: U2.13
- new net CD/DAT3: J3.2, R12.1, U2.29
- new net CLK: J3.5, R14.1, U2.30
- new net CMD: J3.3, R13.1, U2.37
- new net DAT0: J3.7, R11.1, U2.31
- new net D_N: J1.D-, U4.4
- new net D_P: J1.D+, U4.3
- new net ESP32_RX: U2.34, U4.21
- new net ESP32_TX: U2.35, U4.20
- new net LED1: R16.2, U2.10
- new net LED2: R6.2, U2.11
- new net LED3: R4.2, U2.12
- new net LED4: R1.2, U2.13
- new net SD_INSERTED: J3.A, R15.1, U2.33
- new net VBUS: C12.1, J1.VCC, R7.2, U3.3
- net +3V3: now also C14.1, C15.1, C4.1, J3.4, R11.2, R12.2, R13.2, R14.2, R15.2, R24.2, U3.2, U3.4, U4.5, U4.6, U4.7; no longer R1.2, R2.2, R46.2
- net DTR: now also Q1.G, Q2.S, U4.23; no longer Q3.E, R7.2, U21.2
- net EN: now also EN.S1, EN.S2, Q1.D; no longer Q2.C, R4.2
- net EXT_RXD: now also J4.2; no longer J2.2
- net EXT_TXD: now also J4.3; no longer J2.3
- net GND: now also C12.2, C14.2, C15.2, D1.C, D2.C, D3.C, D4.C, EN.P1, EN.P2, IO0.P1, IO0.P2, J3.6, J3.B, J3.MOUNT0, J3.MOUNT1, J3.MOUNT2, J3.MOUNT3, J4.5, J4.SH1, J4.SH2, R8.1, U3.1, U4.2, U4.25; no longer C10.1, C8.1, SW1.P1, SW1.P2, SW2.P1, SW2.P2, U21.18, U21.21, U21.25, U21.26, U21.7
- net IO0: now also IO0.S1, IO0.S2, Q2.D; no longer Q3.C, R6.2
- net N$1: now also J4.1, J4.4, J4.6; no longer J2.1, J2.4
- net N$37: now also R2.1; no longer R32.1
- net N$4: now also D2.A, R4.1; no longer LED1.C, U21.22
- net N$5: now also D3.A, R6.1; no longer LED2.C, U21.23
- net N$6: now also D4.A, R16.1; no longer C8.2, R4.1, SW1.S1, SW1.S2
- net N$7: now also R24.1, U4.9; no longer LED1.A, R1.1
- net N$8: now also R7.1, R8.2, U4.8; no longer LED2.A, R2.1
- net N$9: now also C13.1, U4.16; no longer Q2.B, R7.1
- net N$94: now also D1.A, R1.1; no longer LED6.A, R46.1
- net RTS: now also Q1.S, Q2.G, U4.19; no longer Q2.E, R8.2, U21.3
- net RXD: now also U2.27; no longer U2.35, U21.5
- net SPEAKER: now also R2.2; no longer R32.2
- net TXD: now also U2.28; no longer U2.34, U21.1
Routing:
- net GND: track 16.7 -> 327.0 mm, vias 0 -> 17
- net +3V3: track 3.77 -> 193.3 mm, vias 0 -> 7
- net IO0: track 0.00 -> 44.0 mm, vias 0 -> 4
- net SD_INSERTED: track 0.00 -> 39.4 mm, vias 0 -> 2
- net CMD: track 0.00 -> 36.5 mm, vias 0 -> 2
- net DAT0: track 0.00 -> 35.3 mm, vias 0 -> 2
- net LED1: track 0.00 -> 34.7 mm
- net EN: track 0.00 -> 34.2 mm, vias 0 -> 2
- net LED2: track 0.00 -> 32.3 mm
- net ESP32_RX: track 0.00 -> 30.8 mm, vias 0 -> 2
- net CLK: track 0.00 -> 30.0 mm, vias 0 -> 2
- net ESP32_TX: track 0.00 -> 29.9 mm, vias 0 -> 2
- net LED3: track 0.00 -> 27.9 mm
- net LED4: track 0.00 -> 24.3 mm
- net CD/DAT3: track 0.00 -> 23.2 mm, vias 0 -> 2
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- added copper zone on layer 1, net GND
- added copper zone on layer 16, net GND
Other:
- board size 100 x 50 mm -> 70 x 50 mm
- board text added: "Designed by Kinoshita(@_nosita)"
- board text added: "ReiwaHouse"
- board text added: "Remote RS232C Controller rev.1"

Commit message: [add]add all
Parts:
- moved C1 30.0 mm to (51.4, 37.1)
- moved C3 30.0 mm to (52.9, 30.1)
- moved J4 30.0 mm to (60.5, 25.0)
- moved C7 30.0 mm to (7.70, 33.8)
- moved R24 30.0 mm to (17.7, 26.9)
- moved R3 30.0 mm to (7.70, 36.8)
- moved R5 30.0 mm to (16.7, 38.8)
- moved R8 30.0 mm to (9.70, 27.5)
- moved C11 30.0 mm to (47.2, 37.1)
- moved C12 30.0 mm to (4.60, 20.4)
- moved C2 30.0 mm to (49.3, 37.1)
- moved C5 30.0 mm to (22.1, 42.0)
- moved C9 30.0 mm to (55.0, 30.1)
- moved D1 30.0 mm to (17.5, 2.70)
- moved D2 30.0 mm to (14.5, 2.70)
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Routing:
- net GND: vias 17 -> 241
