File: RemoteSerialController/remoteserialcontroller.sch (EAGLE design)
At the start: 37 parts, among them J1 ZX62R-AB-5P, J2 D-SUB9, Q2 MMSS8050-L, Q3 MMSS8050-L, SW1 SKRPACE010, SW2 SKRPACE010, U1 ADM3202ARUZ, U2 ESP-WROOM-32, U21 FT232RL

Commit message: [fin]finish design
Parts:
- removed C10, C8: 1000pF, taki-library:C-EUC0603
- removed J2: D-SUB9, taki-library:D-SUB9
- removed LED1: RX, taki-library:LEDCHIPLED_0603
- removed LED2: TX, taki-library:LEDCHIPLED_0603
- removed LED6: LED1, taki-library:LEDCHIPLED_0603
- removed Q3: MMSS8050-L, taki-library:MMSS8050-L
- removed R32, R46: 1k, taki-library:R-EU_R0603
- removed SW1, SW2: SKRPACE010, taki-library:SKRPACE010
- removed U21: FT232RL, taki-library:FT232RL
- added C12, C15: 0.1uF, taki-library:C-EUC0603
- added C14: 5uF, taki-library:C-EUC0603
- added D1, D2, D3, D4: B, taki-library:LEDCHIPLED_0603
- added EN, IO0: SKRPACE010, taki-library:SKRPACE010
- added J3: DM3AT-SF-PEJM5, taki-library:DM3AT-SF-PEJM5
- added J4: XM3B-0942-132L, taki-library:XM3B-0942-132L
- added Q1: BSS138, taki-library:BSS138
- added R11, R12, R13, R14, R15, R24: 10k, taki-library:R-EU_R0603
- added R16: 1k, taki-library:R-EU_R0603
- added U3: ADP3338AKCZ-3.3, taki-library:ADP3338AKCZ-3.3
- added U4: CP2104, taki-library:CP2104
- C13: value 0.1uF -> 4.7uF
- C4: value 0.1uF -> 1uF
- Q2: value MMSS8050-L -> BSS138; device taki-library:MMSS8050-L -> taki-library:BSS138
- R4, R6: value 470 -> 1k
- R7: value 10k -> 24k
- R8: value 10k -> 47k
Connections:
- removed net D1_M: J1.D-, U21.USBDM
- removed net D1_P: J1.D+, U21.USBDP
- removed net N$10: Q3.B, R8.1
- removed net N$12: C10.2, R6.1, SW2.S, SW2.S1
- removed net N$50: LED6.C, U2.IO32
- removed net N$84: C13.1, U21.3V3OUT, U21.VCCIO
- removed net N$85: C4.1, J1.VBUS, U21.VCC
- removed net SCL: U2.IO22
- removed net SDA: U2.IO21
- removed net SQW: U2.IO34
- removed net SW3: U2.IO26
- removed net SW4: U2.IO27
- removed net SW5: U2.IO14
- new net CD/DAT3: J3.DATA3-CD/CS_N, R12.1, U2.IO5
- new net CLK: J3.CLK, R14.1, U2.IO18
- new net CMD: J3.CMD/MOSI, R13.1, U2.IO23
- new net DAT0: J3.DATA0/MISO, R11.1, U2.IO19
- new net D_N: J1.D-, U4.D-
- new net D_P: J1.D+, U4.D+
- new net ESP32_RX: U2.RXD0, U4.TXD
- new net ESP32_TX: U2.TXD0, U4.RXD
- new net LED1: R16.2, U2.IO25
- new net LED2: R6.2, U2.IO26
- new net LED3: R4.2, U2.IO27
- new net LED4: R1.2, U2.IO14
- new net SD_INSERTED: J3.A, R15.1, U2.IO21
- new net VBUS: C12.1, J1.VBUS, R7.2, U3.IN
- net +3V3: now also C14.1, C15.1, C4.1, J3.VCC, R11.2, R12.2, R13.2, R14.2, R15.2, R24.2, U3.OUT, U4.REGIN, U4.VDD, U4.VIO; no longer R1.2, R2.2, R46.2
- net DTR: now also Q1.G, Q2.S, U4.DTR; no longer Q3.E, R7.2, U21.!DTR
- net EN: now also EN.S, EN.S1, Q1.D; no longer Q2.C, R4.2
- net EXT_RXD: now also J4.2; no longer J2.2
- net EXT_TXD: now also J4.3; no longer J2.3
- net GND: now also C12.2, C14.2, C15.2, D1.C, D2.C, D3.C, D4.C, EN.P, EN.P1, IO0.P, IO0.P1, J3.B, J3.GND, J4.5, J4.G1, J4.G2, R8.1, U3.GND, U4.GND; no longer C10.1, C8.1, SW1.P, SW1.P1, SW2.P, SW2.P1, U21.GND, U21.GND@1, U21.GND@2, U21.GND@A, U21.TEST
- net IO0: now also IO0.S, IO0.S1, Q2.D; no longer Q3.C, R6.2
- net N$1: now also J4.1, J4.4, J4.6; no longer J2.1, J2.4
- net N$37: now also R2.1; no longer R32.1
- net N$4: now also D2.A, R4.1; no longer LED1.C, U21.CBUS1
- net N$5: now also D3.A, R6.1; no longer LED2.C, U21.CBUS0
- net N$6: now also D4.A, R16.1; no longer C8.2, R4.1, SW1.S, SW1.S1
- net N$7: now also R24.1, U4.RST; no longer LED1.A, R1.1
- net N$8: now also R7.1, R8.2, U4.VBUS; no longer LED2.A, R2.1
- net N$9: now also C13.1, U4.VPP; no longer Q2.B, R7.1
- net N$94: now also D1.A, R1.1; no longer LED6.A, R46.1
- net RTS: now also Q1.S, Q2.G, U4.RTS; no longer Q2.E, R8.2, U21.!RTS
- net RXD: now also U2.IO16; no longer U2.TXD0, U21.RXD
- net SPEAKER: now also R2.2; no longer R32.2
- net TXD: now also U2.IO17; no longer U2.RXD0, U21.TXD
Other:
- moved on the sheet: C1, C11, C13, C2, C3, C4, C7, C9, J1, R1, R10, R2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

Commit message: [update]update schematic and add BOM
Other:
- note added: "Designed by Kinoshita(@_nosita)"
- moved on the sheet: C1, C11, C12, C13, C14, C15, C2, C3, C4, C5, C6, C7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
